File: IRLocalization.sch (EAGLE design)
At the start: 14 parts

Commit message: Added notes
Parts:
- R3, R4, R5: value (none) -> 1450
Other:
- note added: "Add mounting holes and small nonpopulated headers for the daisy chain"
Changed lines of the file:
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@@
 <part name="R1" library="resistor" library_urn="urn:adsk.eagle:library:348" deviceset="R-US_" device="R0603" package3d_urn="urn:adsk.eagle:package:26057/1" value="18"/>
 <part name="R2" library="resistor" library_urn="urn:adsk.eagle:library:348" deviceset="R-US_" device="R0603" package3d_urn="urn:adsk.eagle:package:26057/1" value="10k"/>
-<part name="R3" library="resistor" library_urn="urn:adsk.eagle:library:348" deviceset="R-US_" device="R0603" package3d_urn="urn:adsk.eagle:package:26057/1"/>
-<part name="R4" library="resistor" library_urn="urn:adsk.eagle:library:348" deviceset="R-US_" device="R0603" package3d_urn="urn:adsk.eagle:package:26057/1"/>
-<part name="R5" library="resistor" library_urn="urn:adsk.eagle:library:348" deviceset="R-US_" device="R0603" package3d_urn="urn:adsk.eagle:package:26057/1"/>
+<part name="R3" library="resistor" library_urn="urn:adsk.eagle:library:348" deviceset="R-US_" device="R0603" package3d_urn="urn:adsk.eagle:package:26057/1" value="1450"/>
+<part name="R4" library="resistor" library_urn="urn:adsk.eagle:library:348" deviceset="R-US_" device="R0603" package3d_urn="urn:adsk.eagle:package:26057/1" value="1450"/>
+<part name="R5" library="resistor" library_urn="urn:adsk.eagle:library:348" deviceset="R-US_" device="R0603" package3d_urn="urn:adsk.eagle:package:26057/1" value="1450"/>
 <part name="U$1" library="IR_Localization" deviceset="NMOS_SOT23" device=""/>
 <part name="SUPPLY1" library="supply2" library_urn="urn:adsk.eagle:library:372" deviceset="GND" device=""/>
@@
 <sheet>
 <plain>
+<text x="-101.6" y="58.42" size="1.778" layer="91">Add mounting holes and small nonpopulated headers for the daisy chain</text>
+<text x="-99.06" y="-20.32" size="1.778" layer="91">Add mounting holes and small nonpopulated headers for the daisy chain</text>
+<text x="7.62" y="-20.32" size="1.778" layer="91">Add mounting holes and small nonpopulated headers for the daisy chain</text>
+<text x="5.08" y="60.96" size="1.778" layer="91">Add mounting holes and small nonpopulated headers for the daisy chain</text>
 </plain>
 <instances>

Commit message: PCB added
Parts:
- added R6, R7, R8: 1450, resistor:R-US_R0603
- added SV5, SV6, SV7, SV8: (no value), con-lstb:MA03-1
- added U$5, U$6, U$7: PHOTOTRANSISTOR_2.54, IR_Localization:PHOTOTRANSISTOR_2.54
Connections:
- removed net !RESET: SV1.3, SV2.13, SV3.13, SV4.3
- new net !RESET_1: SV2.13, SV3.13
- new net !RESET_2: SV1.3, SV4.3
- net 3V3: now also SV5.1, SV6.1, SV7.1, SV8.1, U$5.C, U$6.C, U$7.C
- net A0: now also R8.2, U$7.E; no longer R3.2, U$2.E
- net A1: now also R3.2, U$2.E; no longer R4.2, U$3.E
- net A2: now also R7.2, U$6.E; no longer R5.2, U$4.E
- net A3: now also R4.2, U$3.E
- net A4: now also R6.2, U$5.E
- net A5: now also R5.2, U$4.E
- net D10: now also SV6.3
- net D11: now also SV7.3
- net D12: now also SV8.3
- net D9: now also SV5.3
- net GND: now also R6.1, R7.1, R8.1, SV5.2, SV6.2, SV7.2, SV8.2
Other:
- moved on the sheet: R3, R4, R5

Commit message: Added mounting holes
Parts:
- added H1, H2, H3: MOUNT-PAD-ROUND5.5, holes:MOUNT-PAD-ROUND5.5
Connections:
- net N$2 renamed LED+
- net N$4 renamed LED-
- net GND: now also H1.MOUNT, H2.MOUNT, H3.MOUNT
Changed lines of the file:
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@@
 <part name="U$6" library="IR_Localization" deviceset="PHOTOTRANSISTOR_2.54" device=""/>
 <part name="U$7" library="IR_Localization" deviceset="PHOTOTRANSISTOR_2.54" device=""/>
+<part name="H1" library="holes" library_urn="urn:adsk.eagle:library:237" deviceset="MOUNT-PAD-ROUND" device="5.5" package3d_urn="urn:adsk.eagle:package:14291/1"/>
+<part name="H2" library="holes" library_urn="urn:adsk.eagle:library:237" deviceset="MOUNT-PAD-ROUND" device="5.5" package3d_urn="urn:adsk.eagle:package:14291/1"/>
+<part name="H3" library="holes" library_urn="urn:adsk.eagle:library:237" deviceset="MOUNT-PAD-ROUND" device="5.5" package3d_urn="urn:adsk.eagle:package:14291/1"/>
+<part name="SUPPLY14" library="supply2" library_urn="urn:adsk.eagle:library:372" deviceset="GND" device=""/>
+<part name="SUPPLY15" library="supply2" library_urn="urn:adsk.eagle:library:372" deviceset="GND" device=""/>
+<part name="SUPPLY16" library="supply2" library_urn="urn:adsk.eagle:library:372" deviceset="GND" device=""/>
 </parts>
 <sheets>
@@
 <instance part="U$6" gate="G$1" x="127" y="25.4" smashed="yes"/>
 <instance part="U$7" gate="G$1" x="152.4" y="25.4" smashed="yes"/>
+<instance part="H1" gate="G$1" x="-15.24" y="76.2" smashed="yes">
+<attribute name="NAME" x="-12.446" y="76.7842" size="1.778" layer="95"/>
+<attribute name="VALUE" x="-12.446" y="73.7362" size="1.778" layer="96"/>
+</instance>
+<instance part="H2" gate="G$1" x="27.94" y="76.2" smashed="yes">
+<attribute name="NAME" x="30.734" y="76.7842" size="1.778" layer="95"/>
+<attribute name="VALUE" x="30.734" y="73.7362" size="1.778" layer="96"/>
+</instance>
+<instance part="H3" gate="G$1" x="66.04" y="76.2" smashed="yes">
+<attribute name="NAME" x="68.834" y="76.7842" size="1.778" layer="95"/>
+<attribute name="VALUE" x="68.834" y="73.7362" size="1.778" layer="96"/>
+</instance>
+<instance part="SUPPLY14" gate="GND" x="-20.32" y="71.12" smashed="yes">
+<attribute name="VALUE" x="-22.225" y="67.945" size="1.778" layer="96"/>
+</instance>
+<instance part="SUPPLY15" gate="GND" x="22.86" y="71.12" smashed="yes">
+<attribute name="VALUE" x="20.955" y="67.945" size="1.778" layer="96"/>
+</instance>
+<instance part="SUPPLY16" gate="GND" x="60.96" y="71.12" smashed="yes">
+<attribute name="VALUE" x="59.055" y="67.945" size="1.778" layer="96"/>
+</instance>
 </instances>
 <busses>
 </busses>
 <nets>
-<net name="N$2" class="0">
+<net name="LED+" class="0">
 <segment>
 <pinref part="LED1" gate="G$1" pin="A"/>
 <pinref part="R1" gate="G$1" pin="1"/>
 <wire x1="5.08" y1="30.48" x2="5.08" y2="33.02" width="0.1524" layer="91"/>
+<label x="5.08" y="30.48" size="1.778" layer="95"/>
 </segment>
 </net>
@@
 <wire x1="152.4" y1="2.54" x2="152.4" y2="0" width="0.1524" layer="91"/>
 </segment>
+<segment>
+<pinref part="SUPPLY14" gate="GND" pin="GND"/>
+<wire x1="-20.32" y1="73.66" x2="-20.32" y2="76.2" width="0.1524" layer="91"/>
+<pinref part="H1" gate="G$1" pin="MOUNT"/>
+<wire x1="-20.32" y1="76.2" x2="-17.78" y2="76.2" width="0.1524" layer="91"/>
+</segment>
+<segment>
+<pinref part="H2" gate="G$1" pin="MOUNT"/>
+<wire x1="25.4" y1="76.2" x2="22.86" y2="76.2" width="0.1524" layer="91"/>
+<pinref part="SUPPLY15" gate="GND" pin="GND"/>
+<wire x1="22.86" y1="76.2" x2="22.86" y2="73.66" width="0.1524" layer="91"/>
+</segment>
+<segment>
+<pinref part="SUPPLY16" gate="GND" pin="GND"/>
+<wire x1="60.96" y1="73.66" x2="60.96" y2="76.2" width="0.1524" layer="91"/>
+<pinref part="H3" gate="G$1" pin="MOUNT"/>
+<wire x1="60.96" y1="76.2" x2="63.5" y2="76.2" width="0.1524" layer="91"/>
+</segment>
 </net>
-<net name="N$4" class="0">
+<net name="LED-" class="0">
 <segment>
 <pinref part="U$1" gate="G$1" pin="D"/>
 <pinref part="LED1" gate="G$1" pin="C"/>
 <wire x1="5.08" y1="20.32" x2="5.08" y2="22.86" width="0.1524" layer="91"/>
+<label x="5.08" y="20.32" size="1.778" layer="95"/>
 </segment>
 </net>

Commit message: Fixed orientation for nano headers
Connections:
- net A0: now also R4.2, U$3.E; no longer R8.2, U$7.E
- net A1: now also R5.2, U$4.E; no longer R3.2, U$2.E
- net A2: now also R3.2, U$2.E; no longer R7.2, U$6.E
- net A3: now also R8.2, U$7.E; no longer R4.2, U$3.E
- net A5: now also R7.2, U$6.E; no longer R5.2, U$4.E
Changed lines of the file:
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@@
 </segment>
 <segment>
-<pinref part="R8" gate="G$1" pin="2"/>
-<pinref part="U$7" gate="G$1" pin="E"/>
-<wire x1="152.4" y1="17.78" x2="152.4" y2="15.24" width="0.1524" layer="91"/>
-<wire x1="152.4" y1="15.24" x2="152.4" y2="12.7" width="0.1524" layer="91"/>
-<wire x1="152.4" y1="15.24" x2="154.94" y2="15.24" width="0.1524" layer="91"/>
-<junction x="152.4" y="15.24"/>
-<label x="154.94" y="15.24" size="1.778" layer="95" xref="yes"/>
+<wire x1="53.34" y1="15.24" x2="55.88" y2="15.24" width="0.1524" layer="91"/>
+<label x="55.88" y="15.24" size="1.27" layer="95" xref="yes"/>
+<pinref part="R4" gate="G$1" pin="2"/>
+<wire x1="53.34" y1="12.7" x2="53.34" y2="15.24" width="0.1524" layer="91"/>
+<pinref part="U$3" gate="G$1" pin="E"/>
+<wire x1="53.34" y1="17.78" x2="53.34" y2="15.24" width="0.1524" layer="91"/>
+<junction x="53.34" y="15.24"/>
 </segment>
 </net>
@@
 </segment>
 <segment>
-<wire x1="27.94" y1="15.24" x2="30.48" y2="15.24" width="0.1524" layer="91"/>
-<label x="30.48" y="15.24" size="1.27" layer="95" xref="yes"/>
-<pinref part="R3" gate="G$1" pin="2"/>
-<wire x1="27.94" y1="12.7" x2="27.94" y2="15.24" width="0.1524" layer="91"/>
-<pinref part="U$2" gate="G$1" pin="E"/>
-<wire x1="27.94" y1="17.78" x2="27.94" y2="15.24" width="0.1524" layer="91"/>
-<junction x="27.94" y="15.24"/>
+<wire x1="78.74" y1="15.24" x2="81.28" y2="15.24" width="0.1524" layer="91"/>
+<label x="81.28" y="15.24" size="1.27" layer="95" xref="yes"/>
+<pinref part="R5" gate="G$1" pin="2"/>
+<wire x1="78.74" y1="12.7" x2="78.74" y2="15.24" width="0.1524" layer="91"/>
+<pinref part="U$4" gate="G$1" pin="E"/>
+<wire x1="78.74" y1="17.78" x2="78.74" y2="15.24" width="0.1524" layer="91"/>
+<junction x="78.74" y="15.24"/>
 </segment>
 </net>
@@
 </segment>
 <segment>
-<pinref part="R7" gate="G$1" pin="2"/>
-<pinref part="U$6" gate="G$1" pin="E"/>
-<wire x1="127" y1="17.78" x2="127" y2="15.24" width="0.1524" layer="91"/>
-<wire x1="127" y1="15.24" x2="127" y2="12.7" width="0.1524" layer="91"/>
-<wire x1="127" y1="15.24" x2="129.54" y2="15.24" width="0.1524" layer="91"/>
-<junction x="127" y="15.24"/>
-<label x="129.54" y="15.24" size="1.778" layer="95" xref="yes"/>
+<wire x1="27.94" y1="15.24" x2="30.48" y2="15.24" width="0.1524" layer="91"/>
+<label x="30.48" y="15.24" size="1.27" layer="95" xref="yes"/>
+<pinref part="R3" gate="G$1" pin="2"/>
+<wire x1="27.94" y1="12.7" x2="27.94" y2="15.24" width="0.1524" layer="91"/>
+<pinref part="U$2" gate="G$1" pin="E"/>
+<wire x1="27.94" y1="17.78" x2="27.94" y2="15.24" width="0.1524" layer="91"/>
+<junction x="27.94" y="15.24"/>
 </segment>
 </net>
@@
 </segment>
 <segment>
-<wire x1="53.34" y1="15.24" x2="55.88" y2="15.24" width="0.1524" layer="91"/>
-<label x="55.88" y="15.24" size="1.27" layer="95" xref="yes"/>
-<pinref part="R4" gate="G$1" pin="2"/>
-<wire x1="53.34" y1="12.7" x2="53.34" y2="15.24" width="0.1524" layer="91"/>
-<pinref part="U$3" gate="G$1" pin="E"/>
-<wire x1="53.34" y1="17.78" x2="53.34" y2="15.24" width="0.1524" layer="91"/>
-<junction x="53.34" y="15.24"/>
+<pinref part="R8" gate="G$1" pin="2"/>
+<pinref part="U$7" gate="G$1" pin="E"/>
+<wire x1="152.4" y1="17.78" x2="152.4" y2="15.24" width="0.1524" layer="91"/>
+<wire x1="152.4" y1="15.24" x2="152.4" y2="12.7" width="0.1524" layer="91"/>
+<wire x1="152.4" y1="15.24" x2="154.94" y2="15.24" width="0.1524" layer="91"/>
+<junction x="152.4" y="15.24"/>
+<label x="154.94" y="15.24" size="1.778" layer="95" xref="yes"/>
 </segment>
 </net>
@@
 </segment>
 <segment>
-<wire x1="78.74" y1="15.24" x2="81.28" y2="15.24" width="0.1524" layer="91"/>
-<label x="81.28" y="15.24" size="1.27" layer="95" xref="yes"/>
-<pinref part="R5" gate="G$1" pin="2"/>
-<wire x1="78.74" y1="12.7" x2="78.74" y2="15.24" width="0.1524" layer="91"/>
-<pinref part="U$4" gate="G$1" pin="E"/>
-<wire x1="78.74" y1="17.78" x2="78.74" y2="15.24" width="0.1524" layer="91"/>
-<junction x="78.74" y="15.24"/>
+<pinref part="R7" gate="G$1" pin="2"/>
+<pinref part="U$6" gate="G$1" pin="E"/>
+<wire x1="127" y1="17.78" x2="127" y2="15.24" width="0.1524" layer="91"/>
+<wire x1="127" y1="15.24" x2="127" y2="12.7" width="0.1524" layer="91"/>
+<wire x1="127" y1="15.24" x2="129.54" y2="15.24" width="0.1524" layer="91"/>
+<junction x="127" y="15.24"/>
+<label x="129.54" y="15.24" size="1.778" layer="95" xref="yes"/>
 </segment>
 </net>
